File: hardware/radio.sch (KiCad schematic (older format))
At the start: 73 parts, among them J1 JCLK, P2 JLED1, P3 JCEL, U1 G144A12, U2 NCP1117ST18T3G

Commit message: Partially routed schematic.
Parts:
- removed RPU1, RPU2: 1k, Resistors_SMD:R_0603, symbol R
- CRPI1: footprint Pin_Headers:Pin_Header_Straight_2x20 -> pin20x2:PIN_20X2
- LVIN1, LVOUT1: footprint LEDs:LED-0603 -> LEDs:LED-0805
- U1: footprint (none) -> qfn88:qfn88
- XMEM1: footprint Pin_Headers:Pin_Header_Straight_2x22 -> Socket_Strips:Socket_Strip_Straight_2x22
Connections:
- net labels added: VCC5V0
- wire segments 482 -> 481
- no-connect marks 7 -> 5
Changed lines of the file:
@@
 F 0 "U1" H 1640 7840 60  0000 C CNN
 F 1 "G144A12" H 2210 7840 60  0000 C CNN
-F 2 "" H 1550 7900 60  0001 C CNN
+F 2 "qfn88:qfn88" H 1550 7900 60  0001 C CNN
 F 3 "" H 1550 7900 60  0000 C CNN
 	1    1550 7900
@@
 F 0 "U1" H 1640 10490 60  0000 C CNN
 F 1 "G144A12" H 2210 10490 60  0000 C CNN
-F 2 "" H 1550 10550 60  0001 C CNN
+F 2 "qfn88:qfn88" H 1550 10550 60  0001 C CNN
 F 3 "" H 1550 10550 60  0000 C CNN
 	2    1550 10550
@@
 F 0 "U1" H 6790 8490 60  0000 C CNN
 F 1 "G144A12" H 7360 8490 60  0000 C CNN
-F 2 "" H 6700 8550 60  0001 C CNN
+F 2 "qfn88:qfn88" H 6700 8550 60  0001 C CNN
 F 3 "" H 6700 8550 60  0000 C CNN
 	5    6700 8550
@@
 F 0 "CRPI1" H 11150 5600 50  0000 C CNN
 F 1 "RPI_BPLUS_GPIO" H 11950 3975 50  0000 C CNB
-F 2 "Pin_Headers:Pin_Header_Straight_2x20" H 11750 4350 60  0001 C CNN
+F 2 "pin20x2:PIN_20X2" H 11750 4350 60  0001 C CNN
 F 3 "" H 11750 4350 60  0000 C CNN
 	1    11050 3550
@@
 F 0 "U1" H 1840 3840 60  0000 C CNN
 F 1 "G144A12" H 2410 3840 60  0000 C CNN
-F 2 "" H 1750 3900 60  0001 C CNN
+F 2 "qfn88:qfn88" H 1750 3900 60  0001 C CNN
 F 3 "" H 1750 3900 60  0000 C CNN
 	3    1750 3900
@@
 Text Label 2800 3300 2    60   ~ 0
 GPIO_17_L
+Text Label 2800 3600 2    60   ~ 0
+GPIO_22_L
 Text Label 2800 3400 2    60   ~ 0
-GPIO_22_L
+GPIO_18_L
 Text Label 2800 3500 2    60   ~ 0
-GPIO_18_L
-Text Label 2800 3600 2    60   ~ 0
 GPIO_23_L
 Text Label 2800 3700 2    60   ~ 0
@@
 Text Label 6050 3300 2    60   ~ 0
 GPIO_17_H
+Text Label 6050 3600 2    60   ~ 0
+GPIO_22_H
 Text Label 6050 3400 2    60   ~ 0
-GPIO_22_H
+GPIO_18_H
 Text Label 6050 3500 2    60   ~ 0
-GPIO_18_H
-Text Label 6050 3600 2    60   ~ 0
 GPIO_23_H
 Text Label 6050 3700 2    60   ~ 0
@@
 F 0 "XMEM1" H 4700 5950 50  0000 C CNN
 F 1 "XMEM" V 4500 7100 50  0000 C CNN
-F 2 "Pin_Headers:Pin_Header_Straight_2x22" H 4500 6200 60  0001 C CNN
+F 2 "Socket_Strips:Socket_Strip_Straight_2x22" H 4500 6200 60  0001 C CNN
 F 3 "" H 4500 6200 60  0000 C CNN
 	1    4500 7100
@@
 F 0 "LVIN1" H 8250 8050 50  0000 C CNN
 F 1 "LED" H 8250 7850 50  0000 C CNN
-F 2 "LEDs:LED-0603" H 8250 7950 60  0001 C CNN
+F 2 "LEDs:LED-0805" H 8250 7950 60  0001 C CNN
 F 3 "" H 8250 7950 60  0000 C CNN
 	1    8250 7950
@@
 F 0 "LVOUT1" H 10100 8100 50  0000 C CNN
 F 1 "LED" H 10100 7900 50  0000 C CNN
-F 2 "LEDs:LED-0603" H 10100 8000 60  0001 C CNN
+F 2 "LEDs:LED-0805" H 10100 8000 60  0001 C CNN
 F 3 "" H 10100 8000 60  0000 C CNN
 	1    10100 8000
@@
 	12950 2600 13600 2600
 Wire Wire Line
+	1950 3600 3950 3600
+Wire Wire Line
 	1950 3400 3950 3400
 Wire Wire Line
 	1950 3500 3950 3500
 Wire Wire Line
-	1950 3600 3950 3600
-Wire Wire Line
 	1950 3700 3950 3700
 Wire Wire Line
@@
 	5450 3300 6100 3300
 Wire Wire Line
+	5450 3600 6100 3600
+Wire Wire Line
 	5450 3400 6100 3400
 Wire Wire Line
 	5450 3500 6100 3500
-Wire Wire Line
-	5450 3600 6100 3600
 Wire Wire Line
 	5450 3700 6100 3700
@@
 	8100 7650 8100 7550
 Wire Notes Line
-	1800 550  14450 550
+	1800 550  14400 550
 Wire Notes Line
 	14400 550  14400 5600
@@
 	2550 1600 2550 1550
 Connection ~ 2550 1550
-NoConn ~ 12950 1600
-NoConn ~ 12950 1700
 Wire Wire Line
 	10100 8250 10100 8200
@@
 REFCLK1_L
 Text GLabel 3400 4600 0    39   BiDi ~ 0
-REFCLK1_L
+REFCLK2_L
 NoConn ~ 12950 3400
 NoConn ~ 12950 3500
@@
 F 0 "U1" H 11540 8240 60  0000 C CNN
 F 1 "G144A12" H 12110 8240 60  0000 C CNN
-F 2 "" H 11450 8300 60  0001 C CNN
+F 2 "qfn88:qfn88" H 11450 8300 60  0001 C CNN
 F 3 "" H 11450 8300 60  0000 C CNN
 	4    11450 8300
@@
 	7550 8050 7550 8000
 Connection ~ 7550 8000
-$Comp
-L R RPU1
-U 1 1 541A15CA
-P 7850 2500
-F 0 "RPU1" V 7900 2800 40  0000 C CNN
-F 1 "1k" V 7857 2501 40  0000 C CNN
-F 2 "Resistors_SMD:R_0603" V 7780 2500 30  0001 C CNN
-F 3 "" H 7850 2500 30  0000 C CNN
-	1    7850 2500
-	0    1    -1   0
-$EndComp
-Text Label 7000 2500 0    60   ~ 0
-SCL1_H
 Text Label 7000 2900 0    60   ~ 0
 SPI_MISO_H
@@
 Text Label 7000 3200 0    60   ~ 0
 SPI_SCLK_H
-Text Label 7000 2600 0    60   ~ 0
-SDA1_H
 Text Label 7000 2700 0    60   ~ 0
 TXD0_H
@@
 GPIO_13_H
 Wire Wire Line
-	7600 2500 6950 2500
-Wire Wire Line
-	7600 2600 6950 2600
-Wire Wire Line
 	7600 2700 6950 2700
 Wire Wire Line
@@
 Text Label 7000 4600 0    60   ~ 0
 REFCLK2_H
-$Comp
-L R RPU2
-U 1 1 541A315F
-P 7850 2600
-F 0 "RPU2" V 7900 2900 40  0000 C CNN
-F 1 "1k" V 7857 2601 40  0000 C CNN
-F 2 "Resistors_SMD:R_0603" V 7780 2600 30  0001 C CNN
-F 3 "" H 7850 2600 30  0000 C CNN
-	1    7850 2600
-	0    1    -1   0
-$EndComp
 $Comp
 L R RPU3
@@
 	8300 4600 8100 4600
 Wire Wire Line
-	8300 2500 8300 4700
-Wire Wire Line
 	8100 4500 8300 4500
-Connection ~ 8300 4600
 Wire Wire Line
 	8100 4400 8300 4400
 Connection ~ 8300 4500
-Wire Wire Line
-	8300 2500 8100 2500
 Connection ~ 8300 4400
-Wire Wire Line
-	8100 2600 8300 2600
-Connection ~ 8300 2600
 Wire Wire Line
 	8300 2700 8100 2700
@@
 	8100 4300 8300 4300
 Connection ~ 8300 4300
-$Comp
-L GND #PWR026
-U 1 1 541A763F
-P 8300 4700
-F 0 "#PWR026" H 8300 4700 30  0001 C CNN
-F 1 "GND" H 8300 4630 30  0001 C CNN
-F 2 "" H 8300 4700 60  0000 C CNN
-F 3 "" H 8300 4700 60  0000 C CNN
-	1    8300 4700
-	-1   0    0    -1
-$EndComp
 $Comp
 L GS2 XRST1
@@
 $EndComp
 Connection ~ 6600 3900
+Wire Wire Line
+	12950 1700 13350 1700
+Wire Wire Line
+	12950 1600 13350 1600
+Wire Wire Line
+	13350 1600 13350 1700
+Text Label 13350 1600 2    60   ~ 0
+VCC5V0
+Wire Wire Line
+	8300 1100 8300 4600
+Connection ~ 8300 1100
 $EndSCHEMATC

Commit message: Totally rework how the pull up resistors work.
Connections:
- wire segments 481 -> 475
Other:
- moved on the sheet: CDO1, CSYNC1, P3

Commit message: Minor fixes.
Changed lines of the file:
@@
 GPIO_16_H
 NoConn ~ 10900 3400
+Text Label 6050 4600 2    60   ~ 0
+GPIO_06_H
+Text Label 6050 4500 2    60   ~ 0
+GPIO_12_H
+Text Label 6050 4300 2    60   ~ 0
+GPIO_16_H
 Text Label 6050 4200 2    60   ~ 0
-GPIO_06_H
-Text Label 6050 4300 2    60   ~ 0
-GPIO_12_H
-Text Label 6050 4500 2    60   ~ 0
-GPIO_16_H
-Text Label 6050 4600 2    60   ~ 0
 GPIO_19_H
 Text Label 6050 4400 2    60   ~ 0
@@
 Text Label 2450 4550 2    60   ~ 0
 SPI_CE1_L
-Text Label 3900 4200 2    60   ~ 0
+Text Label 3900 4600 2    60   ~ 0
 GPIO_06_L
-Text Label 3900 4300 2    60   ~ 0
+Text Label 3900 4500 2    60   ~ 0
 GPIO_12_L
 Text Label 3900 4400 2    60   ~ 0
 GPIO_13_L
-Text Label 3900 4500 2    60   ~ 0
+Text Label 3900 4300 2    60   ~ 0
 GPIO_16_L
-Text Label 3900 4600 2    60   ~ 0
+Text Label 3900 4200 2    60   ~ 0
 GPIO_19_L
 Text Label 2250 6150 2    60   ~ 0
@@
 Text GLabel 1900 4550 0    39   BiDi ~ 0
 SPI_CE1_L
-Text GLabel 3400 4200 0    39   BiDi ~ 0
+Text GLabel 3400 4600 0    39   BiDi ~ 0
 GPIO_06_L
-Text GLabel 3400 4300 0    39   BiDi ~ 0
+Text GLabel 3400 4500 0    39   BiDi ~ 0
 GPIO_12_L
 Text GLabel 3400 4400 0    39   BiDi ~ 0
 GPIO_13_L
-Text GLabel 3400 4500 0    39   BiDi ~ 0
+Text GLabel 3400 4300 0    39   BiDi ~ 0
 GPIO_16_L
-Text GLabel 3400 4600 0    39   BiDi ~ 0
+Text GLabel 3400 4200 0    39   BiDi ~ 0
 GPIO_19_L
 Text Label 11500 4950 2    60   ~ 0
@@
 	5450 3700 7600 3700
 Wire Wire Line
+	5450 4600 7600 4600
+Wire Wire Line
+	5450 4500 7600 4500
+Wire Wire Line
+	5450 4400 7600 4400
+Wire Wire Line
+	5450 4300 7600 4300
+Wire Wire Line
 	5450 4200 7600 4200
 Wire Wire Line
-	5450 4300 7600 4300
-Wire Wire Line
-	5450 4400 7600 4400
-Wire Wire Line
-	5450 4500 7600 4500
-Wire Wire Line
-	5450 4600 7600 4600
+	3400 4600 3950 4600
+Wire Wire Line
+	3400 4500 3950 4500
+Wire Wire Line
+	3400 4400 3950 4400
+Wire Wire Line
+	3400 4300 3950 4300
 Wire Wire Line
 	3400 4200 3950 4200
 Wire Wire Line
-	3400 4300 3950 4300
-Wire Wire Line
-	3400 4400 3950 4400
-Wire Wire Line
-	3400 4500 3950 4500
-Wire Wire Line
-	3400 4600 3950 4600
-Wire Wire Line
 	4700 5100 4700 5150

Commit message: Adding SPI flash and changing the SPI setup.
Parts:
- removed XSPI1: XSPI, Pin_Headers:Pin_Header_Straight_1x04, symbol CONN_01X04
- added JSPI1: JSPI, symbol CONN_02X02
- added JSPI_WP1: JSPI_WP, symbol CONN_01X02
- added RSPI_WP1: RSPI_WP, symbol R
- added U?: AT45DB041E, SOIC8, symbol AT45DB041E
- added XSPI1: XSPI, symbol CONN_02X04
Connections:
- net labels added: SPI_CLK, SPI_GR_~CE, SPI_MISO, SPI_MOSI, SPI_RPI_~CE, SPI_~CE, VCC
- wire segments 475 -> 641
Other:
- note added: "C"
- note added: "External"
- note added: "GND"
- note added: "GR"
- note added: "GREEN<->RPI"
- note added: "GREEN<->SPI"
- note added: "I"
- note added: "O"
- note added: "OO\nOO"
- note added: "RPI"
- note added: "SPI"
- note added: "SPI<->RPI"
- note added: "VCC"
- note added: "~E"
- moved on the sheet: C1, CDO1, CSYNC1, R4, U1C, ULVL1, XSERDES1

Commit message: Temporary commit with latest updated.
Parts:
- removed CADC1: CADC, Pin_Headers:Pin_Header_Straight_2x08, symbol CONN_02X08
- added CON?: BARREL_JACK, symbol BARREL_JACK
- added CVOUT5 (x2): C, SMD_Packages:SMD-0603, symbol C
- added P? (x3): SATA, symbol SATA
- added P?: CONN_01X03, symbol CONN_01X03
- added U5V0: NCP1117ST33T3G, symbol NCP1117ST33T3G
- added U?: MPCIE-Socket, symbol MPCIE-Socket
- renumbered CVIN1 to CVIN3, CVOUT1 to CVOUT3, U2 to U3V3
Connections:
- net labels added: +5V
- net labels removed: 709.ai, 713.ai, 717.ai, ARX1_617.ai
- wire segments 641 -> 664
- no-connect marks 5 -> 3
Other:
- note added: "A pins == analog in (RX)\nB pins == analog out (TX)"
- moved on the sheet: ARX1, ATX1, CRX1, CTX1, LRX1, RRX1, RRX2, RTX1

Commit message: Removing the antenna from the radio schematic.
Parts:
- removed ARX1: ANTENNA_RX, Connect:bnc, symbol CONN_01X02
- removed ATX1: ANTENNA_TX, Connect:bnc, symbol CONN_01X02
- removed CRX1: C, SMD_Packages:SMD-0603, symbol C
- removed CTX1: 320pF, SMD_Packages:SMD-0603, symbol C
- removed LRX1: 160nH, SMD_Packages:SMD-0603, symbol INDUCTOR
- removed P?: SATA, symbol SATA
- removed RRX1, RRX2: 1k, Resistors_SMD:R_0603, symbol R
- removed RTX1: 50, Resistors_SMD:R_0603, symbol R
Connections:
- wire segments 664 -> 638
Other:
- note added: "Analog Interface"
- note added: "SATA connectors\nA pins == analog in (RX)\nB pins == analog out (TX)"
- note removed: "A pins == analog in (RX)\nB pins == analog out (TX)"
- note removed: "Radio Interface"
- note removed: "Receive Antenna"
- note removed: "Transmit Antenna"
- moved on the sheet: JSPI1, JSPI_WP1, P?, RSPI_WP1, U?, XSPI1

Commit message: Preparing to hook up mPCIe connector and adding documentation.
Connections:
- wire segments 638 -> 526
Other:
- note added: "2 pins - SMB Bus - I2C?"
- note added: "2 pins - USB"
- note added: "5 pins - UIM..."
- note added: "5V"
- note added: "Mini PCI Express has the following;\n\nPower\n * +3.3V - 2 pins\n * +3.3Vaux - 5 pins\n * +1.5V - 3 pins\n * GND - 12 pins\n\nPCI Express - 6 pins\nUSB - 2 pins\nAux - 5 pins (SMB Bus == 2 pins)\nLED - 3 pins\nUIM - 5 pins\n\n---------------------------------\n\nFor GreenArrays memory needs the following;\n\nADDR - 20 pins\nDATA - 18 pins\nCE + WE - 2 pins\n\nTotal: 40 pins (plus power)\n\n------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"
- moved on the sheet: C3, C4, C5, CON?, CVIN3, CVOUT3, CVOUT5, J1, LRST1, LVIN1, LVOUT1, P?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

Commit message: Lots of different fixes.
 * Removing mpcie and replacing with onboard memory (freeing up some pins).

 * Changing the SPI configuration (don't actually need the fancy 3 way header).
   Added lots of documentation how to work with SPI flash for booting,
   programming, etc.

 * Fixed all the electrical DRC errors.
Parts:
- removed JSPI1: JSPI, symbol CONN_02X02
- removed P3: JCEL, Pin_Headers:Pin_Header_Straight_1x03, symbol CONN_01X03
- removed P? (x2): SATA, symbol SATA
- removed U?: MPCIE-Socket, symbol MPCIE-Socket
- removed XMEM1: XMEM, Socket_Strips:Socket_Strip_Straight_2x22, symbol CONN_02X22
- added AN0: Analog 709 / 713, symbol Custom-SATA-Output
- added AN1: Analog 617 / 117, symbol Custom-SATA-Output
- added JFLA_CE1: Flash Chip Enable, symbol CONN_01X02
- added JGNBT1: GA SPI Boot Disable, symbol CONN_01X02
- added RFLA_CE1, RGNBT1: 1k, symbol R
- added RLB1, ROE1, RUB1: 1K, symbol R
- added XMEM1: IS62/65WV51216E(A|B)LL, symbol IS62/65WV51216E(A|B)LL
- JFLA_WP1: renamed from JSPI_WP1; value JSPI_WP -> Flash Write Enable
- RFLA_WP1: renamed from RSPI_WP1; value RSPI_WP -> 1k
- gave numbers to parts that had none: 3
- renumbered CVIN3 to CVIN33, CVOUT5 to CVIN5V0, CVOUT3 to CVOUT1V8, CVOUT5 to CVOUT3V3, LVOUT1 to L1V8, LVIN1 to L3V3, RVOUT1 to RL1V8, RVIN1 to RL3V3, U3V3 to U3V3t1V8, U5V0 to U5V0t3V3
Connections:
- net labels added: 117.ai, 117.ao, 617.ai, 617.ao, 709.ai, 713.ai, 717.ai, ADDRN18, DATA[0..15], JFLA_CE, RST
- net labels removed: ADDRN0, ADDRN19, ATX1_117.ao, DATA16, DATA17, DATA[0..17], GPIO_05_L, SPI_CE1_L, SPI_GR_~CE, SPI_RPI_~CE, VCC
- wire segments 526 -> 491
Other:
- note added: "512Kx16 SRAM"
- note added: "When Green Array boots;\n * It is a SPI master.\n * If 705.17 (SPI_MISO) is high, it won't boot and pins are \n in weak pull-down.\n * If 705.17 (SPI_MISO) is low, looks for SPI device.\n\nJumpering JGNBT1 causes SPI_MISO to have a weak pull up.\nThis disables the GreenArray from booting using SPI. \nDoing this enables operating the flash via either RPi\nor an external programmer.\n\nJumpering JF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"
- note removed: "2 pins - SMB Bus - I2C?"
- note removed: "2 pins - USB"
- note removed: "5 pins - UIM..."
- note removed: "5V"
- note removed: "External"
- note removed: "GR"
- note removed: "GREEN<->RPI"
- note removed: "GREEN<->SPI"
- note removed: "Mini PCI Express has the following;\n\nPower\n * +3.3V - 2 pins\n * +3.3Vaux - 5 pins\n * +1.5V - 3 pins\n * GND - 12 pins\n\nPCI Express - 6 pins\nUSB - 2 pins\nAux - 5 pins (SMB Bus == 2 pins)\nLED - 3 pins\nUIM - 5 pins\n\n---------------------------------\n\nFor GreenArrays memory needs the following;\n\nADDR - 20 pins\nDATA - 18 pins\nCE + WE - 2 pins\n\nTotal: 40 pins (plus power)\n\n------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"
- note removed: "OO\nOO"
- note removed: "RPI"
- note removed: "SPI"
- note removed: "SPI<->RPI"
- moved on the sheet: CVIN5V0, CVOUT3V3, JFLA_WP1, L3V3, RFLA_WP1, RL3V3
