File: hardware/radio.sch (KiCad schematic (older format))
At the start: 85 parts, among them J1 JCLK, U1 G144A12, U3V3t1V8 NCP1117ST18T3G, U5V0t3V3 NCP1117ST33T3G

Commit message: Fixing the values of the 1.8V connected LEDs.
Parts:
- RL1V8, RRST2: value 1k -> 100
Changed lines of the file:
@@
 P 7575 7575
 F 0 "RRST2" V 7655 7575 40  0000 C CNN
-F 1 "1k" V 7582 7576 40  0000 C CNN
+F 1 "100" V 7582 7576 40  0000 C CNN
 F 2 "rsmd:R_0603" V 7505 7575 30  0001 C CNN
 F 3 "" H 7575 7575 30  0000 C CNN
@@
 P 10275 8625
 F 0 "RL1V8" V 10355 8625 40  0000 C CNN
-F 1 "1k" V 10282 8626 40  0000 C CNN
+F 1 "100" V 10282 8626 40  0000 C CNN
 F 2 "rsmd:R_0603" V 10205 8625 30  0001 C CNN
 F 3 "" H 10275 8625 30  0000 C CNN

Commit message: Fixing resistor values.
Parts:
- RL3V3: value 1.5k -> 1k
- RLED1, RLED2, RLED3, RRST1: value 1k -> 100
- renumbered CVIN33 to CVIN3V3
Changed lines of the file:
@@
 P 7825 6675
 F 0 "RRST1" V 7905 6675 40  0000 C CNN
-F 1 "1k" V 7832 6676 40  0000 C CNN
+F 1 "100" V 7832 6676 40  0000 C CNN
 F 2 "rsmd:R_0603" V 7755 6675 30  0001 C CNN
 F 3 "" H 7825 6675 30  0000 C CNN
@@
 $EndComp
 $Comp
-L C-RESCUE-radio CVIN33
+L C-RESCUE-radio CVIN3V3
 U 1 1 541406A2
 P 8825 7975
-F 0 "CVIN33" V 8950 7900 40  0000 L CNN
+F 0 "CVIN3V3" V 8950 7900 40  0000 L CNN
 F 1 "10uF" V 8800 7775 40  0000 L CNN
 F 2 "SMD_Packages:SMD-0805" H 8863 7825 30  0001 C CNN
@@
 P 4250 10100
 F 0 "RLED1" V 4330 10100 40  0000 C CNN
-F 1 "1k" V 4257 10101 40  0000 C CNN
+F 1 "100" V 4257 10101 40  0000 C CNN
 F 2 "rsmd:R_0603" V 4180 10100 30  0001 C CNN
 F 3 "" H 4250 10100 30  0000 C CNN
@@
 P 4250 10400
 F 0 "RLED2" V 4330 10400 40  0000 C CNN
-F 1 "1k" V 4257 10401 40  0000 C CNN
+F 1 "100" V 4257 10401 40  0000 C CNN
 F 2 "rsmd:R_0603" V 4180 10400 30  0001 C CNN
 F 3 "" H 4250 10400 30  0000 C CNN
@@
 P 4250 10700
 F 0 "RLED3" V 4330 10700 40  0000 C CNN
-F 1 "1k" V 4257 10701 40  0000 C CNN
+F 1 "100" V 4257 10701 40  0000 C CNN
 F 2 "rsmd:R_0603" V 4180 10700 30  0001 C CNN
 F 3 "" H 4250 10700 30  0000 C CNN
@@
 P 8350 8625
 F 0 "RL3V3" V 8430 8625 40  0000 C CNN
-F 1 "1.5k" V 8357 8626 40  0000 C CNN
+F 1 "1k" V 8357 8626 40  0000 C CNN
 F 2 "rsmd:R_0603" V 8280 8625 30  0001 C CNN
 F 3 "" H 8350 8625 30  0000 C CNN

Commit message: Removing LED on the SPI Chip Enable line.
This LED can't work because we need a pull up via 1k resistor which we can't
replace with 100 ohm as the GreenArray's needs to be able to pull it down.
Parts:
- removed LSPI_CE1: LED, LEDs:LED-0805, symbol LED-RESCUE-radio
- removed RSPI_CE1: 1k, rsmd:R_0603, symbol R-RESCUE-radio
Connections:
- wire segments 482 -> 479
Changed lines of the file:
@@
-$EndComp
-$Comp
-L LED-RESCUE-radio LSPI_CE1
-U 1 1 545DF6F7
-P 17900 1150
-F 0 "LSPI_CE1" H 17675 1200 50  0000 C CNN
-F 1 "LED" H 17900 1050 50  0000 C CNN
-F 2 "LEDs:LED-0805" H 17900 1150 60  0001 C CNN
-F 3 "" H 17900 1150 60  0000 C CNN
-	1    17900 1150
-	1    0    0    -1
-$EndComp
-$Comp
-L R-RESCUE-radio RSPI_CE1
-U 1 1 545E260F
-P 18400 1150
-F 0 "RSPI_CE1" V 18480 1150 40  0000 C CNN
-F 1 "1k" V 18407 1151 40  0000 C CNN
-F 2 "rsmd:R_0603" V 18330 1150 30  0001 C CNN
-F 3 "" H 18400 1150 30  0000 C CNN
-	1    18400 1150
-	0    -1   -1   0
-$EndComp
-$Comp
-L GND #PWR030
-U 1 1 545E4B31
-P 18700 1150
-F 0 "#PWR030" H 18700 1150 30  0001 C CNN
-F 1 "GND" H 18700 1080 30  0001 C CNN
-F 2 "" H 18700 1150 60  0000 C CNN
-F 3 "" H 18700 1150 60  0000 C CNN
-	1    18700 1150
-	0    -1   -1   0
 $EndComp
 $Comp
@@
 	17900 1725 17900 1675
 Wire Wire Line
-	17700 1150 17450 1150
-Connection ~ 17450 1150
-Wire Wire Line
-	18100 1150 18150 1150
-Wire Wire Line
-	18650 1150 18700 1150
-Wire Wire Line
 	13725 6675 13525 6675

Commit message: Renaming J1 to XCLK1 to be consistent with other headers.
Parts:
- renumbered J1 to XCLK1
Changed lines of the file:
@@
 REFCLK2_L
 $Comp
-L CONN_01X02 J1
+L CONN_01X02 XCLK1
 U 1 1 541471A2
 P 12675 8125
-F 0 "J1" H 12575 8025 50  0000 C CNN
+F 0 "XCLK1" H 12575 8025 50  0000 C CNN
 F 1 "JCLK" V 12775 8125 50  0000 C CNN
 F 2 "Pin_Headers:Pin_Header_Straight_1x02" H 12675 8125 60  0001 C CNN
